File: pcb/cheapino-original.kicad_pcb (KiCad board)
At the start: 2 copper layers, 132.5 x 95.1 mm, 65 parts, among them K1 SW_Push, K10 SW_Push, K11 SW_Push, K12 SW_Push, K13 SW_Push, K14 SW_Push, K15 SW_Push, K16 SW_Push, K17 SW_Push, K18 SW_Push, K19 K19, K2 SW_Push, K20 K20, K21 K21, K3 SW_Push, K4 SW_Push, K5 SW_Push, K6 SW_Push, K7 SW_Push, K8 SW_Push, K9 SW_Push, U1 RP2040-Zero

Commit message: Add 6-column (6x3) Cheapino conversion — WIP routing
Adds 6th physical column per half (K19/K20/K21 + D22/D23/D24), extended
outline, and ROW_4-based matrix wiring. Board loads; all new nets connected.
NOT finished: 2 DRC shorts remain to route. See SIX_COLUMN_HANDOFF.md.
Parts:
- removed D22: D22, keebio:Diode-dual
- removed D23: D23, keebio:Diode-dual
- removed D24: D24, keebio:Diode-dual
- removed K19: K19, project_footprints:Kailh_socket_MX_optional_reversible
- removed K20: K20, project_footprints:Kailh_socket_MX_optional_reversible
- removed K21: K21, project_footprints:Kailh_socket_MX_optional_reversible
Routing:
- net ROW_4: track 248.5 -> 53.9 mm, vias 3 -> 1
- net COL_1: track 367.7 -> 229.2 mm, vias 5 -> 2
- net COL_2: track 376.5 -> 261.6 mm, vias 4 -> 3
- net COL_3: track 390.8 -> 355.4 mm, vias 5 -> 2
- net Net-(D24-K): track 32.0 -> 0.00 mm
- net Net-(D23-K): track 32.0 -> 0.00 mm
- net Net-(D22-K): track 32.0 -> 0.00 mm
